File: Haptic-Map/motor_block.kicad_sch (KiCad schematic)
At the start: 10 parts, among them M1 Motor_DC, U1 DRV2605LDGS, U4 AMS1117-3.3

Commit message: i like watching I2C rail my circuit
Parts:
- removed C3: 10uF, symbol Device:C
- removed C4: 15uF, symbol Device:C
- removed R1: 2, symbol Device:R
- removed R2, R3: 10k, symbol Device:R
- removed U4: AMS1117-3.3, Package_TO_SOT_SMD:SOT-223-3_TabPin2, symbol Regulator_Linear:AMS1117-3.3
Connections:
- net VCC: now also C1.2, U1.10 (VDD)
