File: Haptic-Map/Haptic-Map.kicad_sch (KiCad schematic)
At the start: 5 parts, among them U1 ESP32-S3-MINI-1, U2 AMS1117-3.3

Commit message: fixed schematics
Connections:
- net motor_block/SCL is gone; now on net GND: U1.12 (IO8)
- net motor_block/SDA is gone; now on net GND: U1.13 (IO9)
- net motor_block/EN: now also C2.1, U2.3 (VI)
Changed lines of the file:
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@@
 	(paper "A4")
 	(junction
+		(at 38.1 90.17)
+		(diameter 0)
+		(color 0 0 0 0)
+	)
+	(junction
 		(at 148.59 95.25)
 		(diameter 0)
@@
 	)
 	(junction
+		(at 195.58 25.4)
+		(diameter 0)
+		(color 0 0 0 0)
+	)
+	(junction
+		(at 22.86 90.17)
+		(diameter 0)
+		(color 0 0 0 0)
+	)
+	(junction
 		(at 63.5 95.25)
 		(diameter 0)
@@
 	)
 	(junction
+		(at 22.86 95.25)
+		(diameter 0)
+		(color 0 0 0 0)
+	)
+	(junction
 		(at 207.01 113.03)
 		(diameter 0)
@@
 	)
 	(junction
+		(at 22.86 41.91)
+		(diameter 0)
+		(color 0 0 0 0)
+	)
+	(junction
 		(at 161.29 113.03)
 		(diameter 0)
@@
 	)
 	(junction
+		(at 35.56 95.25)
+		(diameter 0)
+		(color 0 0 0 0)
+	)
+	(junction
 		(at 74.93 113.03)
 		(diameter 0)
@@
 	(wire
 		(pts
+			(xy 22.86 25.4) (xy 195.58 25.4)
+		)
+		(stroke
+			(width 0)
+			(type default)
+		)
+	)
+	(wire
+		(pts
 			(xy 148.59 73.66) (xy 148.59 95.25)
 		)
@@
 	(wire
 		(pts
+			(xy 22.86 25.4) (xy 22.86 41.91)
+		)
+		(stroke
+			(width 0)
+			(type default)
+		)
+	)
+	(wire
+		(pts
 			(xy 199.39 25.4) (xy 199.39 27.94)
 		)
@@
 	(wire
 		(pts
+			(xy 52.07 82.55) (xy 52.07 113.03)
+		)
+		(stroke
+			(width 0)
+			(type default)
+		)
+	)
+	(wire
+		(pts
+			(xy 50.8 38.1) (xy 226.06 38.1)
+		)
+		(stroke
+			(width 0)
+			(type default)
+		)
+	)
+	(wire
+		(pts
+			(xy 132.08 50.8) (xy 132.08 68.58)
+		)
+		(stroke
+			(width 0)
+			(type default)
+		)
+	)
+	(wire
+		(pts
+			(xy 171.45 71.12) (xy 171.45 90.17)
+		)
+		(stroke
+			(width 0)
+			(type default)
+		)
+	)
+	(wire
+		(pts
+			(xy 111.76 71.12) (xy 111.76 90.17)
+		)
+		(stroke
+			(width 0)
+			(type default)
+		)
+	)
+	(wire
+		(pts
+			(xy 77.47 62.23) (xy 77.47 41.91)
+		)
+		(stroke
+			(width 0)
+			(type default)
+		)
+	)
+	(wire
+		(pts
+			(xy 105.41 41.91) (xy 105.41 60.96)
+		)
+		(stroke
+			(width 0)
+			(type default)
+		)
+	)
+	(wire
+		(pts
+			(xy 151.13 71.12) (xy 143.51 71.12)
+		)
+		(stroke
+			(width 0)
+			(type default)
+		)
+	)
+	(wire
+		(pts
 			(xy 195.58 25.4) (xy 199.39 25.4)
 		)
@@
 	(wire
 		(pts
-			(xy 52.07 82.55) (xy 52.07 113.03)
-		)
-		(stroke
-			(width 0)
-			(type default)
-		)
-	)
-	(wire
-		(pts
-			(xy 50.8 38.1) (xy 226.06 38.1)
-		)
-		(stroke
-			(width 0)
-			(type default)
-		)
-	)
-	(wire
-		(pts
-			(xy 132.08 50.8) (xy 132.08 68.58)
-		)
-		(stroke
-			(width 0)
-			(type default)
-		)
-	)
-	(wire
-		(pts
-			(xy 171.45 71.12) (xy 171.45 90.17)
-		)
-		(stroke
-			(width 0)
-			(type default)
-		)
-	)
-	(wire
-		(pts
-			(xy 111.76 71.12) (xy 111.76 90.17)
-		)
-		(stroke
-			(width 0)
-			(type default)
-		)
-	)
-	(wire
-		(pts
-			(xy 77.47 62.23) (xy 77.47 41.91)
-		)
-		(stroke
-			(width 0)
-			(type default)
-		)
-	)
-	(wire
-		(pts
-			(xy 105.41 41.91) (xy 105.41 60.96)
-		)
-		(stroke
-			(width 0)
-			(type default)
-		)
-	)
-	(wire
-		(pts
-			(xy 151.13 71.12) (xy 143.51 71.12)
-		)
-		(stroke
-			(width 0)
-			(type default)
-		)
-	)
-	(wire
-		(pts
 			(xy 135.89 41.91) (xy 163.83 41.91)
 		)
@@
 	(wire
 		(pts
+			(xy 22.86 90.17) (xy 38.1 90.17)
+		)
+		(stroke
+			(width 0)
+			(type default)
+		)
+	)
+	(wire
+		(pts
 			(xy 187.96 62.23) (xy 194.31 62.23)
 		)
@@
 	(wire
 		(pts
+			(xy 22.86 95.25) (xy 22.86 113.03)
+		)
+		(stroke
+			(width 0)
+			(type default)
+		)
+	)
+	(wire
+		(pts
 			(xy 163.83 60.96) (xy 163.83 68.58)
 		)
@@
 	(wire
 		(pts
+			(xy 22.86 90.17) (xy 22.86 95.25)
+		)
+		(stroke
+			(width 0)
+			(type default)
+		)
+	)
+	(wire
+		(pts
 			(xy 187.96 68.58) (xy 187.96 62.23)
 		)
@@
 	(wire
 		(pts
-			(xy 22.86 52.07) (xy 22.86 113.03)
+			(xy 22.86 52.07) (xy 22.86 90.17)
 		)
 		(stroke
@@
 		)
 		(stroke
+			(width 0)
+			(type default)
+		)
+	)
+	(wire
+		(pts
+			(xy 22.86 95.25) (xy 35.56 95.25)
+		)
+		(stroke

Commit message: i like watching I2C rail my circuit
Parts:
- added R1, R2: 4.7k, symbol Device:R
- added U6: TCA9548AMRGER, Package_DFN_QFN:Texas_RGE0024C_VQFN-24-1EP_4x4mm_P0.5mm_EP2.1x2.1mm, symbol Interface_Expansion:TCA9548AMRGER
Connections:
- net GND: now also U6.18 (A2), U6.22 (A0), U6.23 (A1), U6.9 (GND); no longer U1.12 (IO8), U1.13 (IO9)
- net at C8.1, U1.3 (3V3), U2.2 (VO): now also R1.1, R2.1
- new net SCL: R2.2, U1.12 (IO8), U6.19 (SCL)
- new net SDA: R1.2, U1.13 (IO9), U6.20 (SDA)
- new net motor_block/SCL: U6.11 (SC4)
- new net motor_block/SDA: U6.10 (SD4)
- new net motor_block1/SCL: U6.8 (SC3)
- new net motor_block1/SDA: U6.7 (SD3)
- new net motor_block2/SCL: U6.6 (SC2)
- new net motor_block2/SDA: U6.5 (SD2)
- new net motor_block3/SCL: U6.4 (SC1)
- new net motor_block3/SDA: U6.3 (SD1)
- new net motor_block4/SCL: U6.2 (SC0)
- new net motor_block4/SDA: U6.1 (SD0)
- new net motor_block5/SCL: U6.13 (SC5)
- new net motor_block5/SDA: U6.12 (SD5)

Commit message: steps father hates their son
Parts:
- removed V1: 5v, symbol Simulation_SPICE:VDC
- added P1: USB_C_Plug_USB2.0, symbol Connector:USB_C_Plug_USB2.0
Connections:
- net GND: now also P1.A1 (GND), P1.A12 (GND), P1.B1 (GND), P1.B12 (GND)
- net motor_block/EN: now also P1.A4 (VBUS), P1.A9 (VBUS), P1.B4 (VBUS), P1.B9 (VBUS)
Changed lines of the file:
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@@
+	)
+	(junction
+		(at 22.86 41.91)
+		(diameter 0)
+		(color 0 0 0 0)
 	)
 	(junction
@@
 	)
 	(junction
-		(at 22.86 41.91)
-		(diameter 0)
-		(color 0 0 0 0)
-	)
-	(junction
 		(at 161.29 113.03)
 		(diameter 0)
@@
 	(wire
 		(pts
+			(xy 20.32 173.99) (xy 67.31 173.99)
+		)
+		(stroke
+			(width 0)
+			(type default)
+		)
+	)
+	(wire
+		(pts
 			(xy 22.86 25.4) (xy 22.86 41.91)
 		)
@@
 	(wire
 		(pts
-			(xy 127 130.81) (xy 33.02 130.81)
-		)
-		(stroke
-			(width 0)
-			(type default)
-		)
-	)
-	(wire
-		(pts
 			(xy 132.08 50.8) (xy 132.08 68.58)
 		)
@@
 	(wire
 		(pts
+			(xy 67.31 173.99) (xy 67.31 168.91)
+		)
+		(stroke
+			(width 0)
+			(type default)
+		)
+	)
+	(wire
+		(pts
+			(xy 22.86 41.91) (xy 22.86 100.33)
+		)
+		(stroke
+			(width 0)
+			(type default)
+		)
+	)
+	(wire
+		(pts
 			(xy 22.86 41.91) (xy 54.61 41.91)
 		)
@@
 	(wire
 		(pts
-			(xy 22.86 52.07) (xy 22.86 113.03)
-		)
-		(stroke
-			(width 0)
-			(type default)
-		)
-	)
-	(wire
-		(pts
 			(xy 154.94 151.13) (xy 154.94 152.4)
 		)
@@
 	(wire
 		(pts
+			(xy 33.02 130.81) (xy 127 130.81)
+		)
+		(stroke
+			(width 0)
+			(type default)
+		)
+	)
+	(wire
+		(pts
 			(xy 149.86 130.81) (xy 149.86 73.66)
 		)
@@
 	(wire
 		(pts
+			(xy 22.86 100.33) (xy 20.32 100.33)
+		)
+		(stroke
+			(width 0)
+			(type default)
+		)
+	)
+	(wire
+		(pts
 			(xy 102.87 82.55) (xy 102.87 113.03)
 		)
@@
 	(wire
 		(pts
+			(xy 20.32 100.33) (xy 20.32 173.99)
+		)
+		(stroke
+			(width 0)
+			(type default)
+		)
+	)
+	(wire
+		(pts
 			(xy 74.93 82.55) (xy 74.93 113.03)
 		)
@@
 	(wire
 		(pts
+			(xy 22.86 113.03) (xy 22.86 153.67)
+		)
+		(stroke
+			(width 0)
+			(type default)
+		)
+	)
+	(wire
+		(pts
 			(xy 135.89 41.91) (xy 135.89 60.96)
 		)
@@
 		(pts
 			(xy 71.12 67.31) (xy 71.12 62.23)
+		)
+		(stroke
+			(width 0)
+			(type default)
+		)
+	)
+	(wire
+		(pts
+			(xy 22.86 153.67) (xy 29.21 153.67)
 		)
 		(stroke
@@
 	(label "SCL"
 		(at 224.79 63.5 0)
+		(effects
+			(font
+				(size 1.27 1.27)
+			)
+			(justify left bottom)
+		)
+	)
+	(label "Supply atleast 5v and 1.5A"
+		(at 44.45 142.24 0)
 		(effects
 			(font
@@
 	)
 	(symbol
-		(lib_id "Simulation_SPICE:VDC")
-		(at 22.86 46.99 0)
+		(lib_id "Connector:USB_C_Plug_USB2.0")
+		(at 52.07 153.67 270)
 		(unit 1)
 		(exclude_from_sim no)
@@
 		(dnp no)
 		(fields_autoplaced yes)
-		(property "Reference" "V1"
-			(at 26.67 45.5901 0)
+		(property "Reference" "P1"
+			(at 71.12 152.3999 90)
 			(effects
 				(font
@@
 			)
 		)
-		(property "Value" "5v"
-			(at 26.67 48.1301 0)
+		(property "Value" "USB_C_Plug_USB2.0"
+			(at 71.12 154.9399 90)
 			(effects
 				(font
@@
 		)
 		(property "Footprint" ""
-			(at 22.86 46.99 0)
+			(at 52.07 157.48 0)
 			(effects
 				(font
@@
 			)
 		)
-		(property "Datasheet" "https://ngspice.sourceforge.io/docs/ngspice-html-manual/manual.xhtml#sec_Independent_Sources_for"
-			(at 22.86 46.99 0)
+		(property "Datasheet" "https://www.usb.org/sites/default/files/documents/usb_type-c.zip"
+			(at 52.07 157.48 0)
 			(effects
 				(font
@@
 			)
 		)
-		(property "Description" "Voltage source, DC"
-			(at 22.86 46.99 0)
+		(property "Description" "USB 2.0-only Type-C Plug connector"
+			(at 52.07 153.67 0)
 			(effects
 				(font
@@
 			)
 		)
-		(property "Sim.Pins" "1=+ 2=-"
-			(at 22.86 46.99 0)
-			(effects
-				(font
-					(size 1.27 1.27)
-				)
-				(hide yes)
-			)
-		)
-		(property "Sim.Type" "DC"
-			(at 22.86 46.99 0)
-			(effects
-				(font
-					(size 1.27 1.27)
-				)
-				(hide yes)
-			)
-		)
-		(property "Sim.Device" "V"
-			(at 22.86 46.99 0)
-			(effects
-				(font
-					(size 1.27 1.27)
-				)
-				(justify left)
-				(hide yes)
-			)
-		)
-		(pin "1"
-		)
-		(pin "2"
+		(pin "A7"
+		)
+		(pin "A5"
+		)
+		(pin "B1"
+		)
+		(pin "A6"
+		)
+		(pin "A1"
+		)
+		(pin "S1"
+		)
+		(pin "B9"
+		)
+		(pin "A4"
+		)
+		(pin "A9"
+		)
+		(pin "B12"
+		)
+		(pin "B5"
+		)
+		(pin "A12"
+		)
+		(pin "B4"
 		)
 		(instances
 			(project ""
 				(path "/0a30ebb2-76b1-4531-b534-05893d30a2ff"
-					(reference "V1")
+					(reference "P1")
 					(unit 1)
 				)
